Commit message: luennon 5 jälkeen typoja korjattu

File: src/r3_2020/urdf/r3_2020.urdf (robot description, URDF)
Before this commit: robot r3_2020, 5 links, 4 joints
Links:
- added link sonar1_link, mass 0.030; collision box size=0.01 0.05 0.01; visual box size=0.01 0.05 0.01
Joints:
- removed joint wheel_left_link
- added joint sonar1_joint: type fixed, parent base_link, child sonar1_link, origin xyz=-0.235 0 0.16 rpy=0 0 3.14157, axis 0 0 0
- added joint wheel_left_joint: type continuous, parent base_link, child wheel_left_link, origin xyz=0 0 0 rpy=0 0 0, axis 0 -1 0

Commit message: 0 y negatsonarit suunnillen paikoillaan ja näkyy

File: src/r3_2020/urdf/r3_2020.urdf (robot description, URDF)
Before this commit: robot r3_2020, 6 links, 5 joints
Links:
- added link sonar2_link, mass 0.030; collision box size=0.01 0.05 0.01; visual box size=0.01 0.05 0.01
- added link sonar3_link, mass 0.030; collision box size=0.01 0.05 0.01; visual box size=0.01 0.05 0.01
- added link sonar4_link, mass 0.030; collision box size=0.01 0.05 0.01; visual box size=0.01 0.05 0.01
Joints:
- added joint sonar2_joint: type fixed, parent base_link, child sonar2_link, origin xyz=0.234 0 0.16 rpy=0 0 0, axis 0 0 0
- added joint sonar3_joint: type fixed, parent base_link, child sonar3_link, origin xyz=0 -0.235 0.16 rpy=0 0 -1.57079, axis 0 0 0
- added joint sonar4_joint: type fixed, parent base_link, child sonar4_link, origin xyz=0 0.238 0.16 rpy=0 0 1.57079, axis 0 0 0
